Commit message: test RHP for 5 robots

File: cf_description/urdf/cf5.urdf.xacro (robot description, xacro)
@@ -12,5 +12,5 @@
     </inertial>
     <visual>
-      <origin xyz="0 0 0" rpy="0 0 0" />
+      <origin xyz="0 0 0" rpy="4.71 0 0" />
       <geometry>
         <mesh filename="package://multi_uav_simulator/cf_description/crazyflie2.dae"/>
