Commit message: Issue 9:Support for simulating heterogenous quadrotor swarms.

File: multi_uav_simulator/bigquad_description/bigquad.urdf.xacro (robot description, xacro)
@@ -1,9 +1,9 @@
 <?xml version="1.0"?>
-<robot xmlns:xacro="http://www.ros.org/wiki/xacro" name="hector">
+<robot xmlns:xacro="http://www.ros.org/wiki/xacro" name="bigquad">
     <link name="base_link$(arg robot_id)">
       <visual>
         <origin xyz="0 0 0" rpy="3.142 0 0" />
         <geometry>
-          <mesh filename="package://multi_uav_simulator/hector_description/hector.dae"/>
+          <mesh filename="package://multi_uav_simulator/bigquad_description/bigquad.dae"/>
         </geometry>
       </visual>
